File: Swan40.kicad_pcb (KiCad board)
At the start: 2 copper layers, 268 x 87.1 mm, 92 parts, among them SW1 SW_PUSH, SW10 SW_PUSH, SW11 SW_PUSH, SW12 SW_PUSH, SW13 SW_PUSH, SW14 SW_PUSH, SW15 SW_PUSH, SW16 SW_PUSH, SW17 SW_DPDT_x2, SW18 SW_PUSH, SW19 SW_PUSH, SW2 SW_PUSH, SW20 SW_PUSH, SW21 SW_PUSH, SW22 SW_PUSH, SW23 SW_PUSH, SW24 SW_PUSH, SW25 SW_PUSH, SW26 SW_PUSH, SW27 SW_PUSH, SW28 SW_PUSH, SW29 SW_PUSH, SW3 SW_PUSH, SW30 SW_PUSH, SW31 SW_PUSH, SW32 SW_PUSH, SW33 SW_PUSH, SW34 SW_DPDT_x2, SW35 SW_PUSH, SW36 SW_PUSH, SW37 SW_PUSH, SW38 SW_PUSH, SW39 SW_PUSH, SW4 SW_PUSH, SW40 SW_PUSH, SW41 SW_PUSH, SW42 SW_PUSH, SW5 SW_PUSH, SW6 SW_PUSH, SW7 SW_PUSH, SW8 SW_PUSH, SW9 SW_PUSH, U1 xiao_nrf52840, U2 xiao_nrf52840

Commit message: Updated board outline
Other:
- board size 268 x 87.1 mm -> 268 x 87.4 mm
Changed lines of the file:
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@@
     )
   )
+  (gr_arc (start 154.25 42) (mid 155.133883 42.366117) (end 155.5 43.25)
+    (stroke (width 0.1) (type default)) (layer "Edge.Cuts"))
   (gr_arc (start 292.25 107) (mid 260.78 109.129999) (end 229.25 110)
     (stroke (width 0.1) (type default)) (layer "Edge.Cuts"))
-  (gr_line (start 178.25 63.25) (end 178.25 42)
+  (gr_arc (start 161 43.25) (mid 161.366117 42.366117) (end 162.25 42)
     (stroke (width 0.1) (type default)) (layer "Edge.Cuts"))
-  (gr_line (start 151.75 42) (end 155.5 42)
+  (gr_line (start 178.25 62.75) (end 178.25 43.25)
+    (stroke (width 0.1) (type default)) (layer "Edge.Cuts"))
+  (gr_line (start 153 42) (end 154.25 42)
     (stroke (width 0.1) (type default)) (layer "Edge.Cuts"))
   (gr_line (start 161 83.5) (end 168.25 103.75)
     (stroke (width 0.1) (type default)) (layer "Edge.Cuts"))
+  (gr_arc (start 137 42) (mid 137.883883 42.366117) (end 138.25 43.25)
+    (stroke (width 0.1) (type default)) (layer "Edge.Cuts"))
+  (gr_arc (start 138.75 63.25) (mid 138.396447 63.103553) (end 138.25 62.75)
+    (stroke (width 0.1) (type default)) (layer "Edge.Cuts"))
+  (gr_arc (start 151.75 62.75) (mid 151.603553 63.103553) (end 151.25 63.25)
+    (stroke (width 0.1) (type default)) (layer "Edge.Cuts"))
   (gr_line (start 174 119.75) (end 168.25 103.75)
     (stroke (width 0.1) (type default)) (layer "Edge.Cuts"))
-  (gr_line (start 138.25 63.25) (end 151.75 63.25)
+  (gr_line (start 138.75 63.25) (end 151.25 63.25)
     (stroke (width 0.1) (type default)) (layer "Edge.Cuts"))
-  (gr_line (start 178.25 42) (end 183.25 42)
+  (gr_line (start 179.5 42) (end 181.75 42)
     (stroke (width 0.1) (type default)) (layer "Edge.Cuts"))
-  (gr_line (start 155.5 42) (end 155.5 83.5)
+  (gr_line (start 155.5 43.25) (end 155.5 83.5)
     (stroke (width 0.1) (type default)) (layer "Edge.Cuts"))
-  (gr_arc (start 183.25 42) (mid 243.331396 35.521656) (end 292.25 71)
+  (gr_arc (start 181.75 42) (mid 242.609512 35.125826) (end 292.25 71)
     (stroke (width 0.1) (type default)) (layer "Edge.Cuts"))
   (gr_arc (start 87.25 110) (mid 115.428692 111.737416) (end 142.5 119.75)
     (stroke (width 0.1) (type default)) (layer "Edge.Cuts"))
-  (gr_line (start 151.75 63.25) (end 151.75 42)
+  (gr_line (start 151.75 62.75) (end 151.75 43.25)
     (stroke (width 0.1) (type default)) (layer "Edge.Cuts"))
-  (gr_line (start 138.25 42) (end 138.25 63.25)
+  (gr_line (start 138.25 43.25) (end 138.25 62.75)
     (stroke (width 0.1) (type default)) (layer "Edge.Cuts"))
-  (gr_line (start 161 42) (end 164.75 42)
+  (gr_line (start 162.25 42) (end 163.5 42)
     (stroke (width 0.1) (type default)) (layer "Edge.Cuts"))
   (gr_line (start 292.25 107) (end 292.25 71)
     (stroke (width 0.1) (type default)) (layer "Edge.Cuts"))
-  (gr_line (start 164.75 63.25) (end 164.75 42)
+  (gr_line (start 164.75 62.75) (end 164.75 43.25)
     (stroke (width 0.1) (type default)) (layer "Edge.Cuts"))
-  (gr_line (start 164.75 63.25) (end 178.25 63.25)
+  (gr_line (start 165.25 63.25) (end 177.75 63.25)
     (stroke (width 0.1) (type default)) (layer "Edge.Cuts"))
-  (gr_line (start 161 42) (end 161 83.5)
+  (gr_arc (start 165.25 63.25) (mid 164.896447 63.103553) (end 164.75 62.75)
+    (stroke (width 0.1) (type default)) (layer "Edge.Cuts"))
+  (gr_line (start 161 43.25) (end 161 83.5)
     (stroke (width 0.1) (type default)) (layer "Edge.Cuts"))
   (gr_arc (start 87.25 110) (mid 55.72 109.129999) (end 24.25 107)
     (stroke (width 0.1) (type default)) (layer "Edge.Cuts"))
-  (gr_line (start 138.25 42) (end 133.25 42)
+  (gr_line (start 137 42) (end 134.75 42)
     (stroke (width 0.1) (type default)) (layer "Edge.Cuts"))
   (gr_line (start 24.25 71) (end 24.25 107)
@@
   (gr_line (start 148.25 103.75) (end 155.5 83.5)
     (stroke (width 0.1) (type default)) (layer "Edge.Cuts"))
-  (gr_arc (start 24.25 71) (mid 73.168605 35.521656) (end 133.25 42)
+  (gr_arc (start 151.75 43.25) (mid 152.116117 42.366117) (end 153 42)
+    (stroke (width 0.1) (type default)) (layer "Edge.Cuts"))
+  (gr_arc (start 178.25 62.75) (mid 178.103553 63.103553) (end 177.75 63.25)
+    (stroke (width 0.1) (type default)) (layer "Edge.Cuts"))
+  (gr_arc (start 24.25 71) (mid 73.890486 35.125817) (end 134.75 42)
+    (stroke (width 0.1) (type default)) (layer "Edge.Cuts"))
+  (gr_arc (start 178.25 43.25) (mid 178.616117 42.366117) (end 179.5 42)
     (stroke (width 0.1) (type default)) (layer "Edge.Cuts"))
   (gr_arc (start 174 119.75) (mid 201.071308 111.737416) (end 229.25 110)
     (stroke (width 0.1) (type default)) (layer "Edge.Cuts"))
+  (gr_arc (start 163.5 42) (mid 164.383883 42.366117) (end 164.75 43.25)
+    (stroke (width 0.1) (type default)) (layer "Edge.Cuts"))
   (gr_line (start 142.5 119.75) (end 148.25 103.75)

Commit message: Wiring complete
Parts:
- removed H1, H3: BAT+, kbd:1pin_conn
- removed H2, H4: BAT-, kbd:1pin_conn
- removed TP1, TP3: BOARD+, kbd:1pad_conn_board
- removed TP2, TP4: BOARD-, kbd:1pad_conn_board
- added BAT+: BAT+, kbd:1pad_conn_board, B.Cu at (172.8, 81.5)
- added BAT+: BAT+, kbd:1pad_conn_board, B.Cu at (123.2, 81.5)
- added BAT-: BAT-, kbd:1pad_conn_board, B.Cu at (167.8, 81.5)
- added BAT-: BAT-, kbd:1pad_conn_board, B.Cu at (128.2, 81.5)
- added BRD+: BOARD+, kbd:1pad_conn_board, B.Cu at (132.0, 67.0)
- added BRD+: BOARD+, kbd:1pad_conn_board, B.Cu at (158.5, 67.0)
- added BRD-: BOARD-, kbd:1pad_conn_board, B.Cu at (137.5, 67.0)
- added BRD-: BOARD-, kbd:1pad_conn_board, B.Cu at (164.0, 67.0)
- moved D24 15.7 mm to (163.0, 105.1)
- moved D28 15.7 mm to (183.1, 99.6)
- moved D32 15.7 mm to (203.8, 97.8)
- moved SW25 15.7 mm to (164.8, 109.8)
- moved SW29 15.7 mm to (184.0, 104.5)
- moved SW33 15.7 mm to (203.8, 102.8)
- moved SW17 11.4 mm to (143.5, 75.5)
- moved SW34 11.4 mm to (152.5, 75.5)
- moved D19 10.4 mm to (114.0, 80.9)
- moved SW20 10.4 mm to (114.0, 85.8)
- moved D25 10.3 mm to (200.0, 44.8)
- moved D26 10.3 mm to (200.0, 61.8)
- moved D29 10.3 mm to (218.0, 39.8)
- moved D30 10.3 mm to (218.0, 56.8)
- moved D33 10.3 mm to (236.0, 45.8)
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Routing:
- net RCOL5: track 0.00 -> 192.0 mm
- net RCOL4: track 0.00 -> 191.1 mm
- net LROW4: track 7.45 -> 188.7 mm, vias 5 -> 6
- net RROW4: track 7.37 -> 183.7 mm, vias 5 -> 6
- net LCOL2: track 0.00 -> 154.8 mm
- net RCOL3: track 0.00 -> 153.1 mm, vias 0 -> 2
- net LCOL1: track 0.00 -> 152.1 mm
- net RCOL2: track 0.00 -> 147.5 mm, vias 0 -> 2
- net LROW1: track 7.56 -> 142.8 mm, vias 5 -> 6
- net LROW3: track 7.56 -> 138.5 mm, vias 5 -> 6
- net LROW2: track 7.55 -> 137.9 mm, vias 5 -> 6
- net LCOL3: track 0.00 -> 130.0 mm
- net RCOL1: track 0.00 -> 120.3 mm, vias 0 -> 2
- net RROW3: track 7.39 -> 118.1 mm, vias 5 -> 6
- net RROW1: track 7.39 -> 108.9 mm, vias 5 -> 6
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Other:
- board size 268 x 87.4 mm -> 268 x 89.1 mm
