File: Swan40-rounded.kicad_pcb (KiCad board)
At the start: 2 copper layers, 268 x 89.1 mm, 92 parts, among them SW1 SW_PUSH, SW10 SW_PUSH, SW11 SW_PUSH, SW12 SW_PUSH, SW13 SW_PUSH, SW14 SW_PUSH, SW15 SW_PUSH, SW16 SW_PUSH, SW17 SW_DPDT_x2, SW18 SW_PUSH, SW19 SW_PUSH, SW2 SW_PUSH, SW20 SW_PUSH, SW21 SW_PUSH, SW22 SW_PUSH, SW23 SW_PUSH, SW24 SW_PUSH, SW25 SW_PUSH, SW26 SW_PUSH, SW27 SW_PUSH, SW28 SW_PUSH, SW29 SW_PUSH, SW3 SW_PUSH, SW30 SW_PUSH, SW31 SW_PUSH, SW32 SW_PUSH, SW33 SW_PUSH, SW34 SW_DPDT_x2, SW35 SW_PUSH, SW36 SW_PUSH, SW37 SW_PUSH, SW38 SW_PUSH, SW39 SW_PUSH, SW4 SW_PUSH, SW40 SW_PUSH, SW41 SW_PUSH, SW42 SW_PUSH, SW5 SW_PUSH, SW6 SW_PUSH, SW7 SW_PUSH, SW8 SW_PUSH, SW9 SW_PUSH, U1 xiao_nrf52840, U2 xiao_nrf52840

Commit message: Fixed errors + Rounded tracks
Routing:
- net RCOL5: track 195.1 -> 190.7 mm
- net RCOL4: track 191.3 -> 188.0 mm
- net LCOL2: track 154.7 -> 151.8 mm
- net RCOL1: track 122.0 -> 119.3 mm
- net LCOL3: track 127.3 -> 124.7 mm
- net LROW1: track 142.8 -> 140.7 mm
- net RROW4: track 182.7 -> 180.6 mm
- net RCOL3: track 152.8 -> 150.9 mm
- net RCOL2: track 147.5 -> 145.6 mm
- net LROW2: track 137.8 -> 136.0 mm
- net LCOL4: track 98.4 -> 96.8 mm
- net LROW3: track 134.8 -> 133.3 mm
- net LROW4: track 188.7 -> 187.2 mm
- net RROW3: track 116.9 -> 115.4 mm
- net RROW1: track 108.4 -> 107.1 mm
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
Commit message: Rounded + added droplets + fill zones
Parts:
- added REF**: 0.5mm_hole, kbd:0.5mm_hole, F.Cu at (146.2, 65.0)
- added REF**: 0.5mm_hole, kbd:0.5mm_hole, F.Cu at (146.2, 64.0)
- added REF**: 0.5mm_hole, kbd:0.5mm_hole, F.Cu at (148.8, 97.5)
- added REF**: 0.5mm_hole, kbd:0.5mm_hole, F.Cu at (148.8, 95.5)
- added REF**: 0.5mm_hole, kbd:0.5mm_hole, F.Cu at (148.8, 65.0)
- added REF**: 0.5mm_hole, kbd:0.5mm_hole, F.Cu at (148.8, 68.0)
- added REF**: 0.5mm_hole, kbd:0.5mm_hole, F.Cu at (146.2, 97.5)
- added REF**: 0.5mm_hole, kbd:0.5mm_hole, F.Cu at (146.2, 95.5)
- added REF**: 0.5mm_hole, kbd:0.5mm_hole, F.Cu at (148.8, 94.5)
- added REF**: 0.5mm_hole, kbd:0.5mm_hole, F.Cu at (146.2, 66.0)
- added REF**: 0.5mm_hole, kbd:0.5mm_hole, F.Cu at (148.8, 93.5)
- added REF**: 0.5mm_hole, kbd:0.5mm_hole, F.Cu at (148.8, 67.0)
- added REF**: 0.5mm_hole, kbd:0.5mm_hole, F.Cu at (148.8, 66.0)
- added REF**: 0.5mm_hole, kbd:0.5mm_hole, F.Cu at (146.2, 94.5)
- added REF**: 0.5mm_hole, kbd:0.5mm_hole, F.Cu at (148.8, 64.0)
- added REF**: 0.5mm_hole, kbd:0.5mm_hole, F.Cu at (146.2, 68.0)
- added REF**: 0.5mm_hole, kbd:0.5mm_hole, F.Cu at (146.2, 93.5)
- added REF**: 0.5mm_hole, kbd:0.5mm_hole, F.Cu at (146.2, 67.0)
- added REF**: 0.5mm_hole, kbd:0.5mm_hole, F.Cu at (146.2, 96.5)
- added REF**: 0.5mm_hole, kbd:0.5mm_hole, F.Cu at (148.8, 96.5)
- moved D21 1.25 mm to (180.8, 46.8)
- moved D22 1.25 mm to (180.8, 63.8)
- moved D23 1.25 mm to (180.8, 80.8)
- moved D24 1.25 mm to (161.8, 105.1)
- moved D25 1.25 mm to (198.8, 44.8)
- moved D26 1.25 mm to (198.8, 61.8)
- moved D27 1.25 mm to (198.8, 78.8)
- moved D28 1.25 mm to (181.9, 99.6)
- moved D29 1.25 mm to (216.8, 39.8)
- moved D30 1.25 mm to (216.8, 56.8)
- moved D31 1.25 mm to (216.8, 73.8)
- moved D32 1.25 mm to (202.5, 97.8)
- moved D33 1.25 mm to (234.8, 45.8)
- moved D34 1.25 mm to (234.8, 62.8)
- moved D35 1.25 mm to (234.8, 79.8)
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- renumbered BAT+ to TP1, BAT- to TP2, BRD+ to TP3, BRD- to TP4, BAT+ to TP5, BAT- to TP6, BRD+ to TP7, BRD- to TP8
Connections:
- U1 pad 13: unconnected-(U1-GND-Pad13) -> LGND
- U2 pad 13: unconnected-(U2-GND-Pad13) -> RGND
Routing:
- net Net-(SW17A-B): track 38.0 -> 22.5 mm
- net Net-(SW17A-C): track 43.2 -> 45.4 mm
- net LCOL3: track 124.7 -> 125.7 mm
- added copper zone on B.Cu, net LGND
- added copper zone on F.Cu, net LGND
- added copper zone on B.Cu, net RGND
- added copper zone on F.Cu, net RGND
Other:
- board size 268 x 89.1 mm -> 266.5 x 89.1 mm

Commit message: Added base kibot automation
Parts:
- added REF**: 5mm_hole, kbd:5mm_hole, F.Cu at (171.5, 101.2)
- added REF**: 5mm_hole, kbd:5mm_hole, F.Cu at (123.5, 101.2)
- added REF**: 5mm_hole, kbd:5mm_hole, F.Cu at (189.0, 42.5)
- added REF**: 5mm_hole, kbd:5mm_hole, F.Cu at (262.5, 72.5)
- added REF**: 5mm_hole, kbd:5mm_hole, F.Cu at (32.5, 72.5)
- added REF**: 2.5mm_hole, kbd:2.5mm_hole, F.Cu at (126.0, 67.5)
- added REF**: 2.5mm_hole, kbd:2.5mm_hole, F.Cu at (126.0, 96.0)
- added REF**: 5mm_hole, kbd:5mm_hole, F.Cu at (106.0, 42.5)
- added REF**: 2.5mm_hole, kbd:2.5mm_hole, F.Cu at (169.0, 95.8)
- added REF**: 2.5mm_hole, kbd:2.5mm_hole, F.Cu at (169.0, 67.5)
- moved BAT+ 0.20 mm to (171.5, 81.7)
- moved BAT+ 0.20 mm to (123.5, 81.7)
- moved BAT- 0.20 mm to (166.5, 81.7)
- moved BAT- 0.20 mm to (128.5, 81.7)
- moved BOARD+ 0.20 mm to (132.2, 67.2)
- moved BOARD+ 0.20 mm to (157.2, 67.2)
- moved BOARD- 0.20 mm to (137.8, 67.2)
- moved BOARD- 0.20 mm to (162.8, 67.2)
- moved D1 0.20 mm to (42.0, 58.0)
- moved D10 0.20 mm to (78.2, 57.0)
- moved D11 0.20 mm to (78.2, 74.0)
- moved D12 0.20 mm to (92.5, 98.0)
- moved D13 0.20 mm to (96.3, 45.0)
- moved D14 0.20 mm to (96.2, 62.0)
- moved D15 0.20 mm to (96.3, 79.0)
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- renumbered TP5 to BAT+, TP1 to BAT+, TP6 to BAT-, TP2 to BAT-, TP3 to BOARD+, TP7 to BOARD+, TP4 to BOARD-, TP8 to BOARD-
Routing:
- net LCOL1: track 152.9 -> 150.3 mm
- net RCOL4: track 188.3 -> 186.9 mm
- net RCOL1: track 118.9 -> 120.1 mm
Other:
- outline, holes or cut-outs redrawn

Commit message: Everything re-aligned and re-wired
Parts:
- removed the REF** at (146.2, 65.2)
- removed the REF** at (146.2, 93.7)
- removed the REF** at (146.2, 67.2)
- removed the REF** at (146.2, 96.7)
- removed the REF** at (148.8, 96.7)
- removed the REF** at (146.2, 64.2)
- removed the REF** at (148.8, 97.7)
- removed the REF** at (148.8, 95.7)
- removed the REF** at (148.8, 65.2)
- removed the REF** at (148.8, 68.2)
- removed the REF** at (146.2, 97.7)
- removed the REF** at (146.2, 95.7)
- removed the REF** at (148.8, 94.7)
- removed the REF** at (146.2, 66.2)
- removed the REF** at (148.8, 93.7)
- removed the REF** at (148.8, 66.2)
- removed the REF** at (148.8, 67.2)
- removed the REF** at (146.2, 94.7)
- removed the REF** at (148.8, 64.2)
- removed the REF** at (146.2, 68.2)
- moved BOARD+ 0.58 mm to (131.8, 67.5)
- moved BOARD+ 0.58 mm to (157.8, 67.5)
- moved BOARD- 0.58 mm to (137.2, 67.5)
- moved BOARD- 0.58 mm to (163.2, 67.5)
- moved D13 0.53 mm to (95.8, 45.0)
- moved D15 0.53 mm to (95.8, 79.0)
- moved D20 0.51 mm to (132.7, 105.3)
- moved SW16 0.51 mm to (111.7, 104.8)
- moved SW21 0.50 mm to (131.0, 110.0)
- moved U1 0.50 mm to (134.5, 53.0)
- moved U2 0.50 mm to (160.5, 53.0)
- moved D28 0.50 mm to (182.4, 99.8)
- moved SW29 0.50 mm to (183.3, 104.7)
- moved BAT+ 0.50 mm to (172.0, 81.7)
- moved BAT+ 0.50 mm to (123.0, 81.7)
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Routing:
- net LCOL1: track 150.3 -> 160.5 mm
- net RCOL5: track 190.7 -> 181.5 mm, vias 0 -> 2
- net RCOL2: track 145.5 -> 137.3 mm
- net LROW2: track 136.0 -> 128.1 mm
- net RROW4: track 180.7 -> 188.3 mm, vias 6 -> 5
- net LROW1: track 140.7 -> 146.3 mm
- net RROW3: track 115.4 -> 120.1 mm, vias 6 -> 5
- net LCOL2: track 151.8 -> 154.9 mm
- net RROW1: track 107.1 -> 105.4 mm, vias 6 -> 5
- net LROW3: track 133.3 -> 134.9 mm
- net RROW2: track 104.7 -> 105.8 mm, vias 6 -> 5
- net RCOL4: track 186.9 -> 188.0 mm, vias 0 -> 2
- net RCOL3: track 150.9 -> 152.0 mm
- net LCOL3: track 125.8 -> 124.8 mm
- net Net-(D1-A): track 11.0 -> 11.6 mm
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Other:
- board size 266.5 x 89.1 mm -> 268 x 89.1 mm

Commit message: Added mouse bites
Parts:
- added REF**: 5x3mm_mouse_bite, kbd:5x3mm_mouse_bite, F.Cu at (147.5, 66.2)
- added REF**: 5x3mm_mouse_bite, kbd:5x3mm_mouse_bite, F.Cu at (147.5, 92.5)
Routing:
- net RCOL4: track 188.0 -> 189.9 mm
- net RCOL5: track 181.5 -> 180.0 mm
- net RCOL3: track 152.0 -> 153.1 mm
- net LCOL3: track 124.8 -> 125.9 mm
- net LCOL4: track 97.2 -> 97.9 mm
Other:
- outline, holes or cut-outs redrawn
